File: Diag586220_Harness/Diag586220_User_Port/Rev.0/Eagle/C64_Userport_Test.sch (EAGLE design)
At the start: 18 parts, among them IC1 4066N, IC2 4066N, J1 C64-USERPORT

Commit message: Add files via upload
values from 120k to 110k and 320R to 316R
Parts:
- added TP1, TP2, TP3: L1,2_R, Pads:L1,2_R
- R1, R2, R5, R6: value 120k -> 110k
- R3: value 320R -> 316R
- renumbered BHR1 to DRL1, BHR2 to DRL2
Connections:
- net +5VCTR1: now also TP2.1
- net +5VCTR2: now also TP3.1
- net GND: now also TP1.1
Changed lines of the file:
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@@
 <?xml version="1.0" encoding="utf-8"?>
 <!DOCTYPE eagle SYSTEM "eagle.dtd">
-<eagle version="9.2.2">
+<eagle version="9.5.2">
 <drawing>
 <settings>
@@
 <part name="U$9" library="!pownet" deviceset="+5V" device=""/>
 <part name="R4" library="DISCRETE" deviceset="RES04" device="" value="150R"/>
-<part name="R3" library="DISCRETE" deviceset="RES04" device="" value="320R"/>
+<part name="R3" library="DISCRETE" deviceset="RES04" device="" value="316R"/>
 <part name="U$10" library="!pownet" deviceset="GND" device=""/>
 <part name="R7" library="DISCRETE" deviceset="RES04" device="" value="0R"/>
-<part name="R1" library="DISCRETE" deviceset="RES04" device="" value="120k"/>
-<part name="R2" library="DISCRETE" deviceset="RES04" device="" value="120k"/>
-<part name="R5" library="DISCRETE" deviceset="RES04" device="" value="120k"/>
-<part name="R6" library="DISCRETE" deviceset="RES04" device="" value="120k"/>
+<part name="R1" library="DISCRETE" deviceset="RES04" device="" value="110k"/>
+<part name="R2" library="DISCRETE" deviceset="RES04" device="" value="110k"/>
+<part name="R5" library="DISCRETE" deviceset="RES04" device="" value="110k"/>
+<part name="R6" library="DISCRETE" deviceset="RES04" device="" value="110k"/>
 <part name="U$11" library="!pownet" deviceset="GND" device=""/>
 <part name="U$12" library="!pownet" deviceset="GND" device=""/>
@@
 <part name="C2" library="DISCRETE" deviceset="CAP01" device="" value="100n"/>
 <part name="C3" library="DISCRETE" deviceset="CAP01" device="" value="100n"/>
-<part name="BHR1" library="Mech_Bohr" deviceset="BOHR3,2" device=""/>
-<part name="BHR2" library="Mech_Bohr" deviceset="BOHR3,2" device=""/>
+<part name="DRL1" library="Mech_Bohr" deviceset="BOHR3,2" device=""/>
+<part name="DRL2" library="Mech_Bohr" deviceset="BOHR3,2" device=""/>
+<part name="TP1" library="Pads" deviceset="L1,2_R" device=""/>
+<part name="TP2" library="Pads" deviceset="L1,2_R" device=""/>
+<part name="TP3" library="Pads" deviceset="L1,2_R" device=""/>
+<part name="U$19" library="!pownet" deviceset="GND" device=""/>
 </parts>
 <sheets>
@@
 <attribute name="VALUE" x="209.55" y="59.69" size="1.27" layer="96" rot="R90"/>
 </instance>
-<instance part="BHR1" gate="G$1" x="231.14" y="57.15" smashed="yes">
+<instance part="DRL1" gate="G$1" x="231.14" y="57.15" smashed="yes">
 <attribute name="NAME" x="229.235" y="59.055" size="1.778" layer="95"/>
 </instance>
-<instance part="BHR2" gate="G$1" x="238.76" y="57.15" smashed="yes">
+<instance part="DRL2" gate="G$1" x="238.76" y="57.15" smashed="yes">
 <attribute name="NAME" x="236.855" y="59.055" size="1.778" layer="95"/>
+</instance>
+<instance part="TP1" gate="G$1" x="53.34" y="137.16" smashed="yes">
+<attribute name="NAME" x="50.8" y="142.24" size="1.778" layer="95"/>
+</instance>
+<instance part="TP2" gate="G$1" x="256.54" y="139.7" smashed="yes">
+<attribute name="NAME" x="254" y="144.78" size="1.778" layer="95"/>
+</instance>
+<instance part="TP3" gate="G$1" x="256.54" y="99.06" smashed="yes">
+<attribute name="NAME" x="254" y="104.14" size="1.778" layer="95"/>
+</instance>
+<instance part="U$19" gate="1" x="53.34" y="132.08" smashed="yes">
+<attribute name="VALUE" x="51.1175" y="130.175" size="1.524" layer="96"/>
 </instance>
 </instances>
@@
 <pinref part="U$16" gate="1" pin="GND"/>
 <wire x1="127" y1="35.56" x2="129.54" y2="35.56" width="0.1524" layer="91"/>
+</segment>
+<segment>
+<pinref part="U$19" gate="1" pin="GND"/>
+<pinref part="TP1" gate="G$1" pin="1"/>
+<wire x1="53.34" y1="134.62" x2="53.34" y2="137.16" width="0.1524" layer="91"/>
 </segment>
 </net>
@@
 <label x="236.22" y="149.86" size="1.6764" layer="95"/>
 <label x="236.22" y="139.7" size="1.6764" layer="95"/>
+<pinref part="TP2" gate="G$1" pin="1"/>
+<wire x1="248.92" y1="139.7" x2="256.54" y2="139.7" width="0.1524" layer="91"/>
+<junction x="248.92" y="139.7"/>
 </segment>
 </net>
@@
 <label x="238.76" y="109.22" size="1.6764" layer="95"/>
 <label x="238.76" y="99.06" size="1.6764" layer="95"/>
-</segment>
-</net>
+<pinref part="TP3" gate="G$1" pin="1"/>
+<wire x1="248.92" y1="99.06" x2="256.54" y2="99.06" width="0.1524" layer="91"/>
+<junction x="248.92" y="99.06"/>
+</segment>
+</net>
